File: cockatiel.kicad_pcb (KiCad board)
At the start: 4 copper layers, 51 x 60 mm, 39 parts, among them J1 Programmer, J10 MIC_N_BYP, J11 MIC_P_SEL, J12 MIC_N_SEL, J13 Cox Box Mic In, J14 Cox Box Mic Out, J15 Mic Out, J16 Headset/Mic In, J3 DEBUG_UART, J4 RESET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

Commit message: Swap pin assignment for the battery connector
It seems most Li-Po batteries are wired this way round.
Connections:
- J7 pad 1: +BATT -> Earth
- J7 pad 2: Earth -> +BATT
Other:
- board text added: "+"
- board text added: "-"
Changed lines of the file:
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@@
     (fp_line (start 3.95 6.25) (end 3.95 -1.35) (layer "F.Fab") (width 0.1))
     (pad "1" thru_hole roundrect (at 0 0 180) (size 1.2 1.75) (drill 0.75) (layers *.Cu *.Mask) (roundrect_rratio 0.2083333333)
-      (net 6 "+BATT") (pinfunction "Pin_1") (pintype "passive"))
+      (net 2 "Earth") (pinfunction "Pin_1") (pintype "passive"))
     (pad "2" thru_hole oval (at 2 0 180) (size 1.2 1.75) (drill 0.75) (layers *.Cu *.Mask)
-      (net 2 "Earth") (pinfunction "Pin_2") (pintype "passive"))
+      (net 6 "+BATT") (pinfunction "Pin_2") (pintype "passive"))
     (model "${KICAD6_3DMODEL_DIR}/Connector_JST.3dshapes/JST_PH_S2B-PH-K_1x02_P2.00mm_Horizontal.wrl"
       (offset (xyz 0 0 0))
@@
   (gr_line (start 120.579655 135.754004) (end 120.573965 135.745032) (layer "F.SilkS") (width 0.22))
   (gr_line (start 120.719215 138.196934) (end 120.753653 138.170389) (layer "F.SilkS") (width 0.22))
+  (gr_circle (center 110.5 112) (end 111.2 112) (layer "F.SilkS") (width 0.2) (fill none))
   (gr_line (start 119.954083 135.910233) (end 119.960806 135.906638) (layer "F.SilkS") (width 0.22))
   (gr_line (start 121.47223 135.571065) (end 121.4894 135.574989) (layer "F.SilkS") (width 0.22))
@@
     (effects (font (size 1.5 1) (thickness 0.25) italic))
   )
+  (gr_text "+" (at 110.5 111.9) (layer "F.SilkS")
+    (effects (font (size 1 1) (thickness 0.25)))
+  )
+  (gr_text "-" (at 114.1 111.9) (layer "F.SilkS")
+    (effects (font (size 1 1) (thickness 0.25)))
+  )
   (gr_text "JLCJLCJLCJLC" (at 124 109) (layer "F.SilkS")
